File: synchronus-4-bit-down-counter/7-seg-disp.kicad_sch (KiCad schematic)
At the start: 0 parts

Commit message: finished KiCAD Schematic
Parts:
- added R10, R7, R8, R9: 10k, Resistor_SMD:R_0805_2012Metric_Pad1.20x1.40mm_HandSolder, symbol 000_Resistors_Immo:10k
- added R11, R12, R13, R14, R15, R16, R17: 330r, Resistor_SMD:R_0805_2012Metric_Pad1.20x1.40mm_HandSolder, symbol 000_Resistors_Immo:Resistor_0805
- added SW3: data, symbol Switch:SW_DIP_x04
- added U10: HDSP-5553-7-segment-cc, Display_7Segment:HDSP-7401, symbol 000_Diodes_Immo:HDSP-7401
- added U11, U12, U13, U14, U9: 4071-quad-OR, symbol 000_Logic_IC_Immo:4071-quad-OR
- added U15, U16, U17: 4081-quad-AND, symbol 000_Logic_IC_Immo:4081-quad-AND
- added U7: 4069, symbol 4xxx:4069
Connections:
- new net: U9.1, U9.4
- new net: U9.10, U9.2
- new net: R11.2, U10.10 (A)
- new net: R16.2, U10.2 (F)
- new net: R17.2, U10.3 (G)
- new net: R15.2, U10.4 (E)
- new net: R14.2, U10.5 (D)
- new net: R13.2, U10.8 (C)
- new net: R12.2, U10.9 (B)
- new net: U12.10, U12.2
- new net: U12.11, U12.9
- new net: U13.2, U13.4
- new net: U14.10, U14.2
- new net: U14.1, U14.4
- new net: U13.11, U13.9
- new net: U11.1, U11.4
- new net: U11.10, U11.2
- new net: U12.1, U12.4
- new net 5V: SW3.5, SW3.6, SW3.7, SW3.8, U11.14 (VDD), U12.14 (VDD), U13.14 (VDD), U14.14 (VDD), U15.14 (VDD), U16.14 (VDD), U17.14 (VDD), U7.14 (VDD), U9.14 (VDD)
- new net A: R10.2, SW3.1, U13.1, U17.2, U17.5, U17.8, U7.1
- new net AB: U13.12, U17.4
- new net AC: U14.9, U17.10
- new net A~{B}C: U12.13, U17.3
- new net B: R9.2, SW3.2, U14.5, U15.1, U15.6, U17.6, U7.3
- new net B~{C}: U12.6, U15.3, U9.5
- new net C: SW3.3, U13.6, U15.8, U16.6, U17.9, U7.5
- new net D: R7.2, R8.2, SW3.4, U12.8, U14.6, U16.2, U7.9, U9.8
- new net GND: R10.1, R7.1, R8.1, R9.1, U10.1 (CC/gnd), U10.6 (CC/gnd), U11.7 (VSS), U12.7 (VSS), U13.7 (VSS), U14.7 (VSS), U15.7 (VSS), U16.7 (VSS), U17.7 (VSS), U7.7 (VSS), U9.7 (VSS)
- new net dA: R11.1, U14.3
- new net dB: R12.1, U13.10
- new net dC: R13.1, U13.3
- new net dD: R14.1, U12.3
- new net dE: R15.1, U11.11
- new net dF: R16.1, U11.3
- new net dG: R17.1, U9.3
- new net ~{A}: U15.12, U15.5, U16.5, U16.8, U7.2
- new net ~{A}B: U11.12, U12.5, U15.4, U9.6
- new net ~{A}C: U11.9, U16.4
- new net ~{A}~{B}: U11.6, U13.8, U15.11
- new net ~{A}~{C}: U11.13, U12.12, U14.8, U16.10
- new net ~{B}: U13.5, U15.13, U15.9, U16.1, U7.4
- new net ~{B}C: U11.5, U15.10, U17.1, U9.9
- new net ~{B}D: U11.8, U16.3
- new net ~{C}: U13.13, U15.2, U16.9, U7.6
- new net ~{D}: U7.8

Commit message: xvcbdfb
Connections:
- net A: now also SW3.4, U7.9; no longer SW3.1, U7.1
- net A~{B}C: now also U12.2; no longer U12.13
- net B: now also SW3.3, U7.5; no longer SW3.2, U7.3
- net B~{C}: now also U11.1, U12.9; no longer U12.6, U9.5
- net C: now also SW3.2, U12.13, U7.3; no longer SW3.3, U13.6, U7.5
- net D: now also SW3.1, U11.12, U12.5, U7.1; no longer SW3.4, U12.8, U7.9, U9.8
- net dA: now also U9.10; no longer U14.3
- net dB: now also U9.11; no longer U13.10
- net dD: now also U13.4; no longer U12.3
- net dE: now also U13.10; no longer U11.11
- net dF: now also U9.4; no longer U11.3
- net ~{A}: now also U7.8; no longer U7.2
- net ~{A}B: now also U11.2, U12.8, U13.8; no longer U11.12, U12.5, U9.6
- net ~{A}~{B}: now also U9.12; no longer U13.8
- net ~{A}~{C}: now also U12.1, U13.9; no longer U11.13, U12.12
- net ~{B}: now also U12.12, U7.6; no longer U13.5, U7.4
- net ~{B}C: now also U11.13; no longer U9.9
- net ~{C}: now also U7.4; no longer U7.6
- net ~{D}: now also U7.2; no longer U7.8
- net at U9.1: now also U11.3; no longer U9.4
- net at U9.2: now also U11.11; no longer U9.10
- net at U12.10: now also U13.5; no longer U12.2
- net at U12.11: now also U13.2; no longer U12.9
- net at U14.10: now also U9.9; no longer U14.2
- net at U14.4: now also U9.8; no longer U14.1
- net at U13.11: now also U9.13; no longer U13.9
- net at U11.4: now also U9.5; no longer U11.1
- net at U11.10: now also U9.6; no longer U11.2
- net at U12.4: now also U13.6; no longer U12.1
- new net: U12.3, U12.6
Other:
- moved on the sheet: U14D, U9D

Commit message: drgdegr
Parts:
- renumbered U17 to U16, U16 to U17
Other:
- moved on the sheet: U11A, U15A, U9A

Commit message: fdhfrth
Other:
- moved on the sheet: U14B, U14C, U16C, U9C

Commit message: sdvsdv
Other:
- moved on the sheet: U14A, U14D, U7E, U7F
Changed lines of the file:
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@@
     )
   )
-  (symbol (lib_id "000_Logic_IC_Immo:4071-quad-OR") (at 368.3 212.09 0) (unit 1)
-    (in_bom yes) (on_board yes) (dnp no) (fields_autoplaced)
-    (property "Reference" "U14" (at 368.3 204.47 0)
-      (effects (font (size 1.27 1.27)))
-    )
-    (property "Value" "4071-quad-OR" (at 368.3 207.01 0)
-      (effects (font (size 1.27 1.27)))
-    )
-    (property "Footprint" "" (at 368.3 212.09 0)
-      (effects (font (size 1.27 1.27)) hide)
-    )
-    (property "Datasheet" "http://www.intersil.com/content/dam/Intersil/documents/cd40/cd4071bms-72bms-75bms.pdf" (at 368.3 212.09 0)
+  (symbol (lib_id "000_Logic_IC_Immo:4071-quad-OR") (at 27.305 210.185 0) (unit 1)
+    (in_bom yes) (on_board yes) (dnp no) (fields_autoplaced)
+    (property "Reference" "U14" (at 27.305 202.565 0)
+      (effects (font (size 1.27 1.27)))
+    )
+    (property "Value" "4071-quad-OR" (at 27.305 205.105 0)
+      (effects (font (size 1.27 1.27)))
+    )
+    (property "Footprint" "" (at 27.305 210.185 0)
+      (effects (font (size 1.27 1.27)) hide)
+    )
+    (property "Datasheet" "http://www.intersil.com/content/dam/Intersil/documents/cd40/cd4071bms-72bms-75bms.pdf" (at 27.305 210.185 0)
       (effects (font (size 1.27 1.27)) hide)
     )
@@
     )
   )
-  (symbol (lib_id "000_Logic_IC_Immo:4071-quad-OR") (at 368.3 229.235 0) (unit 4)
-    (in_bom yes) (on_board yes) (dnp no) (fields_autoplaced)
-    (property "Reference" "U14" (at 368.3 220.98 0)
-      (effects (font (size 1.27 1.27)))
-    )
-    (property "Value" "4071-quad-OR" (at 368.3 223.52 0)
-      (effects (font (size 1.27 1.27)))
-    )
-    (property "Footprint" "" (at 368.3 229.235 0)
-      (effects (font (size 1.27 1.27)) hide)
-    )
-    (property "Datasheet" "http://www.intersil.com/content/dam/Intersil/documents/cd40/cd4071bms-72bms-75bms.pdf" (at 368.3 229.235 0)
+  (symbol (lib_id "000_Logic_IC_Immo:4071-quad-OR") (at 27.305 227.33 0) (unit 4)
+    (in_bom yes) (on_board yes) (dnp no) (fields_autoplaced)
+    (property "Reference" "U14" (at 27.305 219.075 0)
+      (effects (font (size 1.27 1.27)))
+    )
+    (property "Value" "4071-quad-OR" (at 27.305 221.615 0)
+      (effects (font (size 1.27 1.27)))
+    )
+    (property "Footprint" "" (at 27.305 227.33 0)
+      (effects (font (size 1.27 1.27)) hide)
+    )
+    (property "Datasheet" "http://www.intersil.com/content/dam/Intersil/documents/cd40/cd4071bms-72bms-75bms.pdf" (at 27.305 227.33 0)
       (effects (font (size 1.27 1.27)) hide)
     )
@@
     )
   )
-  (symbol (lib_id "4xxx:4069") (at 34.925 271.145 0) (unit 5)
-    (in_bom yes) (on_board yes) (dnp no) (fields_autoplaced)
-    (property "Reference" "U7" (at 34.925 262.89 0)
-      (effects (font (size 1.27 1.27)))
-    )
-    (property "Value" "4069" (at 34.925 265.43 0)
-      (effects (font (size 1.27 1.27)))
-    )
-    (property "Footprint" "" (at 34.925 271.145 0)
-      (effects (font (size 1.27 1.27)) hide)
-    )
-    (property "Datasheet" "http://www.intersil.com/content/dam/Intersil/documents/cd40/cd4069ubms.pdf" (at 34.925 271.145 0)
+  (symbol (lib_id "4xxx:4069") (at 25.4 260.35 0) (unit 5)
+    (in_bom yes) (on_board yes) (dnp no) (fields_autoplaced)
+    (property "Reference" "U7" (at 25.4 252.095 0)
+      (effects (font (size 1.27 1.27)))
+    )
+    (property "Value" "4069" (at 25.4 254.635 0)
+      (effects (font (size 1.27 1.27)))
+    )
+    (property "Footprint" "" (at 25.4 260.35 0)
+      (effects (font (size 1.27 1.27)) hide)
+    )
+    (property "Datasheet" "http://www.intersil.com/content/dam/Intersil/documents/cd40/cd4069ubms.pdf" (at 25.4 260.35 0)
       (effects (font (size 1.27 1.27)) hide)
     )
@@
     )
   )
-  (symbol (lib_id "4xxx:4069") (at 22.86 252.73 0) (unit 6)
-    (in_bom yes) (on_board yes) (dnp no) (fields_autoplaced)
-    (property "Reference" "U7" (at 22.86 245.11 0)
-      (effects (font (size 1.27 1.27)))
-    )
-    (property "Value" "4069" (at 22.86 247.65 0)
-      (effects (font (size 1.27 1.27)))
-    )
-    (property "Footprint" "" (at 22.86 252.73 0)
-      (effects (font (size 1.27 1.27)) hide)
-    )
-    (property "Datasheet" "http://www.intersil.com/content/dam/Intersil/documents/cd40/cd4069ubms.pdf" (at 22.86 252.73 0)
-      (effects (font (size 1.27 1.27)) hide)
-    )
+  (symbol (lib_id "4xxx:4069") (at 26.035 242.57 0) (unit 6)
+    (in_bom yes) (on_board yes) (dnp no) (fields_autoplaced)
+    (property "Reference" "U7" (at 26.035 234.95 0)
+      (effects (font (size 1.27 1.27)))
+    )
+    (property "Value" "4069" (at 26.035 237.49 0)
+      (effects (font (size 1.27 1.27)))
+    )
+    (property "Footprint" "" (at 26.035 242.57 0)
+      (effects (font (size 1.27 1.27)) hide)
+    )
+    (property "Datasheet" "http://www.intersil.com/content/dam/Intersil/documents/cd40/cd4069ubms.pdf" (at 26.035 242.57 0)
+      (effects (font (size 1.27 1.27)) hide)
+    )
