File: synchronus-4-bit-down-counter/synchronus-4-bit-down-counter.kicad_sch (KiCad schematic)
At the start: 19 parts, among them SW1 clear, SW2 CLK, U1 4071-quad-OR, U2 4071-quad-OR, U3 4081-quad-AND, U4 4081-quad-AND, U5 4081-quad-AND, U6 4081-quad-AND, U8 74LS175_D-latch

Commit message: finished KiCAD Schematic
Other:
- sheet 7-segment-display ports: added 5V, A, B, C, D, GND; removed none
Changed lines of the file:
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@@
   (junction (at 201.295 245.745) (diameter 0) (color 0 0 0 0)
   )
+  (junction (at 288.925 156.21) (diameter 0) (color 0 0 0 0)
+  )
   (junction (at 253.365 158.115) (diameter 0) (color 0 0 0 0)
   )
@@
   (junction (at 56.515 163.195) (diameter 0) (color 0 0 0 0)
   )
+  (junction (at 280.035 158.75) (diameter 0) (color 0 0 0 0)
+  )
   (junction (at 245.745 245.745) (diameter 0) (color 0 0 0 0)
   )
+  (junction (at 296.545 153.67) (diameter 0) (color 0 0 0 0)
+  )
   (junction (at 50.165 71.755) (diameter 0) (color 0 0 0 0)
   )
@@
   (junction (at 83.185 41.275) (diameter 0) (color 0 0 0 0)
   )
+  (junction (at 270.51 161.29) (diameter 0) (color 0 0 0 0)
+  )
   (junction (at 276.225 276.86) (diameter 0) (color 0 0 0 0)
   )
@@
     (stroke (width 0) (type default))
   )
+  (wire (pts (xy 288.925 156.21) (xy 288.925 173.99))
+    (stroke (width 0) (type default))
+  )
   (wire (pts (xy 194.945 160.655) (xy 209.55 160.655))
     (stroke (width 0) (type default))
@@
     (stroke (width 0) (type default))
   )
-  (wire (pts (xy 296.545 30.48) (xy 296.545 173.99))
+  (wire (pts (xy 296.545 30.48) (xy 296.545 153.67))
     (stroke (width 0) (type default))
   )
@@
     (stroke (width 0) (type default))
   )
+  (wire (pts (xy 280.035 158.75) (xy 318.77 158.75))
+    (stroke (width 0) (type default))
+  )
   (wire (pts (xy 50.165 95.25) (xy 50.165 203.835))
     (stroke (width 0) (type default))
@@
     (stroke (width 0) (type default))
   )
-  (wire (pts (xy 288.925 73.66) (xy 288.925 173.99))
+  (wire (pts (xy 288.925 73.66) (xy 288.925 156.21))
     (stroke (width 0) (type default))
   )
@@
     (stroke (width 0) (type default))
   )
+  (wire (pts (xy 280.035 158.75) (xy 280.035 173.99))
+    (stroke (width 0) (type default))
+  )
   (wire (pts (xy 140.335 147.32) (xy 163.195 147.32))
     (stroke (width 0) (type default))
   )
+  (wire (pts (xy 296.545 153.67) (xy 296.545 173.99))
+    (stroke (width 0) (type default))
+  )
+  (wire (pts (xy 270.51 161.29) (xy 318.77 161.29))
+    (stroke (width 0) (type default))
+  )
   (wire (pts (xy 330.2 224.79) (xy 328.93 224.79))
     (stroke (width 0) (type default))
@@
     (stroke (width 0) (type default))
   )
-  (wire (pts (xy 280.035 110.49) (xy 280.035 173.99))
+  (wire (pts (xy 280.035 110.49) (xy 280.035 158.75))
     (stroke (width 0) (type default))
   )
@@
     (stroke (width 0) (type default))
   )
+  (wire (pts (xy 296.545 153.67) (xy 318.77 153.67))
+    (stroke (width 0) (type default))
+  )
   (wire (pts (xy 163.83 83.185) (xy 157.48 83.185))
     (stroke (width 0) (type default))
   )
+  (wire (pts (xy 384.81 27.305) (xy 384.81 31.115))
+    (stroke (width 0) (type default))
+  )
   (wire (pts (xy 36.83 127) (xy 100.965 127))
     (stroke (width 0) (type default))
@@
     (stroke (width 0) (type default))
   )
+  (wire (pts (xy 288.925 156.21) (xy 318.77 156.21))
+    (stroke (width 0) (type default))
+  )
   (wire (pts (xy 276.225 278.13) (xy 276.225 276.86))
     (stroke (width 0) (type default))
@@
     (stroke (width 0) (type default))
   )
+  (wire (pts (xy 385.445 194.945) (xy 385.445 193.675))
+    (stroke (width 0) (type default))
+  )
   (wire (pts (xy 116.205 152.4) (xy 163.195 152.4))
     (stroke (width 0) (type default))
@@
   )
   (wire (pts (xy 73.025 245.745) (xy 73.025 248.285))
-    (stroke (width 0) (type default))
-  )
-  (wire (pts (xy 404.495 211.455) (xy 400.05 211.455))
     (stroke (width 0) (type default))
   )
@@
     )
   )
+  (symbol (lib_id "power:GND") (at 385.445 194.945 0) (unit 1)
+    (in_bom yes) (on_board yes) (dnp no) (fields_autoplaced)
+    (property "Reference" "#PWR06" (at 385.445 201.295 0)
+      (effects (font (size 1.27 1.27)) hide)
+    )
+    (property "Value" "GND" (at 385.445 200.025 0)
+      (effects (font (size 1.27 1.27)))
+    )
+    (property "Footprint" "" (at 385.445 194.945 0)
+      (effects (font (size 1.27 1.27)) hide)
+    )
+    (property "Datasheet" "" (at 385.445 194.945 0)
+      (effects (font (size 1.27 1.27)) hide)
+    )
+    (pin "1")
+    (instances
+      (project "synchronus-4-bit-down-counter"
+        (path "/e64d16c4-cbfb-4b73-a7ff-c50bb64351f4"
+          (reference "#PWR06") (unit 1)
+        )
+      )
+    )
+  )
   (symbol (lib_id "000_Logic_IC_Immo:74LS175_D-latch") (at 273.685 261.62 0) (unit 5)
     (in_bom yes) (on_board yes) (dnp no) (fields_autoplaced)
@@
     )
   )
+  (symbol (lib_id "power:+5V") (at 384.81 27.305 0) (unit 1)
+    (in_bom yes) (on_board yes) (dnp no) (fields_autoplaced)
+    (property "Reference" "#PWR07" (at 384.81 31.115 0)
+      (effects (font (size 1.27 1.27)) hide)
+    )
+    (property "Value" "+5V" (at 384.81 24.13 0)
+      (effects (font (size 1.27 1.27)))
+    )
+    (property "Footprint" "" (at 384.81 27.305 0)
+      (effects (font (size 1.27 1.27)) hide)
+    )
+    (property "Datasheet" "" (at 384.81 27.305 0)
+      (effects (font (size 1.27 1.27)) hide)
+    )
+    (pin "1")
+    (instances
+      (project "synchronus-4-bit-down-counter"
+        (path "/e64d16c4-cbfb-4b73-a7ff-c50bb64351f4"
+          (reference "#PWR07") (unit 1)
+        )
+      )
+    )
+  )
   (symbol (lib_id "000_Logic_IC_Immo:4081-quad-AND") (at 164.465 230.505 0) (unit 4)
     (in_bom yes) (on_board yes) (dnp no) (fields_autoplaced)
@@
   )
   (sheet (at 318.77 31.115) (size 74.295 162.56) (fields_autoplaced)
-    (stroke (width 0.1524) (type solid))
-    (fill (color 0 0 0 0.0000))
+    (stroke (width 0.1524) (type solid) (color 255 205 44 0.82))
+    (fill (color 56 56 56 0.3300))
     (property "Sheetname" "7-segment-display" (at 318.77 30.4034 0)
       (effects (font (size 1.27 1.27)) (justify left bottom))
@@
       (effects (font (size 1.27 1.27)) (justify left top))
     )
-    (instances
+    (pin "GND" passive (at 385.445 193.675 270)
+      (effects (font (size 1.27 1.27)) (justify left))
+    )
+    (pin "B" input (at 318.77 156.21 180)
+      (effects (font (size 1.27 1.27)) (justify left))
+    )
+    (pin "C" input (at 318.77 158.75 180)
+      (effects (font (size 1.27 1.27)) (justify left))
+    )
+    (pin "D" input (at 318.77 161.29 180)
+      (effects (font (size 1.27 1.27)) (justify left))
+    )
+    (pin "A" input (at 318.77 153.67 180)
+      (effects (font (size 1.27 1.27)) (justify left))
+    )
+    (pin "5V" passive (at 384.81 31.115 90)
+      (effects (font (size 1.27 1.27)) (justify right))
+    )
+    (instances

Commit message: sdvsdv
Other:
- moved on the sheet: R1, R2, SW1, SW2, U8E
